File: hardware/rows-25.10mm/creeper-eyes-rows-25.10mm.kicad_pcb (KiCad board)
At the start: 2 copper layers, 71.7 x 56 mm, 9 parts, among them J3 OLED, Frank's right eye, J4 OLED, Frank's left eye, J5 DS3231 RTC (optional), U1 ESP32 DevKit V1 (30 pin)

Commit message: Rev B: an RTC header the DS3231 mini plugs onto
Rev A's J5 followed the six-pin ZS-042 (32K SQW SCL SDA VCC GND).  The
module actually in use is the five-pin DS3231 mini sold for the
Raspberry Pi, labelled + D C NC -, which needed jumpers.

J5 is now five pins on rows 12-16, VCC SDA SCL NC GND from the top, GND
on the bottom pin.  SCL keeps its route; SDA comes down its column to
row 13 rather than 15, which avoids the row-14 GND run it would
otherwise have to cross; VCC and GND take rows 12 and 16.  Rows 14-18
were tried first and failed DRC on the bottom-right mounting hole.

ERC clean, schematic and board netlists agree on all 51 nodes, DRC
clean, for both row pitches.  Gerbers regenerated.  The hardware README
gains a Revisions section, with the jumper wiring for rev A boards.

Co-Authored-By: Claude Opus 5.5 <noreply@anthropic.com>
Parts:
- J5: footprint Connector_PinHeader_2.54mm:PinHeader_1x06_P2.54mm_Vertical -> Connector_PinHeader_2.54mm:PinHeader_1x05_P2.54mm_Vertical
Connections:
- J5 pad 1: unconnected-(J5-32K-Pad1) -> 3V3
- J5 pad 2: unconnected-(J5-SQW-Pad2) -> SDA
- J5 pad 4: SDA -> unconnected-(J5-NC-Pad4)
- J5 pad 5: 3V3 -> GND
Routing:
- net SDA: track 40.7 -> 35.6 mm
- net 3V3: track 128.1 -> 124.3 mm
- net GND: track 123.0 -> 120.5 mm
Other:
- board text added: "NC"
- board text added: "creeper-eyes carrier rev B rows 25.10 mm"
- board text removed: "32K"
- board text removed: "SQW"
- board text removed: "creeper-eyes carrier rev A rows 25.10 mm"
